Commit message: Modified the robot shape

File: description/robot_core.xacro (robot description, xacro)
@@ -30,5 +30,5 @@
             <origin xyz="0.15 0 0.075"/>
             <geometry>
-                <box size="0.3 0.3 0.15"/>
+                <cylinder radius="0.15" length="0.15" />
             </geometry>
             <material name="white"/>

Commit message: modifed and added some scripts

File: description/robot_core.xacro (robot description, xacro)
@@ -45,10 +45,10 @@
             <origin xyz="0.15 0 0.075"/>
             <geometry>
-                <box size="0.3 0.3 0.15"/>
+                <cylinder radius="0.15" length="0.15" />
             </geometry>
         </collision>
-        <xacro:inertial_box mass="0.5" x="0.3" y="0.3" z="0.15">
+        <xacro:inertial_cylinder mass="0.5" length="0.15" radius="0.15">
             <origin xyz="0.15 0 0.075" rpy="0 0 0"/>
-        </xacro:inertial_box>
+        </xacro:inertial_cylinder>
     </link>
     <gazebo reference="chassis">
@@ -134,3 +134,50 @@
         <mu2 value="0.001"/>
     </gazebo>
+    <!-- BUMBER SENSOR -->
+    <gazebo>
+  <plugin name="bumper_plugin" filename="libgazebo_ros_bumper.so">
+    <ros>
+      <namespace>/</namespace>
+      <remapping>bumper_states:=/bumper</remapping>
+    </ros>
+    <frame_name>base_link</frame_name>
+  </plugin>
+</gazebo>
+<gazebo reference="base_link">
+  <collision name="bumper_collision">
+    <geometry>
+      <box>
+        <size>0.3 0.3 0.1</size>
+      </box>
+    </geometry>
+  </collision>
+</gazebo>
+<!-- IMU Sensor -->
+<link name="imu_link">
+  <inertial>
+    <mass value="0.1"/>
+    <inertia ixx="0.001" ixy="0.0" ixz="0.0"
+             iyy="0.001" iyz="0.0"
+             izz="0.001"/>
+  </inertial>
+</link>
+<joint name="imu_joint" type="fixed">
+  <parent link="base_link"/>
+  <child link="imu_link"/>
+  <origin xyz="0 0 0.05" rpy="0 0 0"/>
+</joint>
+<gazebo reference="imu_link">
+  <sensor name="imu_sensor" type="imu">
+    <always_on>true</always_on>
+    <update_rate>100</update_rate>
+    <topic>imu/data_raw</topic>
+    <plugin filename="libgazebo_ros_imu_sensor.so" name="imu_plugin">
+      <ros>
+        <namespace>/</namespace>
+        <remapping>~/out:=imu/data_raw</remapping>
+      </ros>
+      <initial_orientation_as_reference>true</initial_orientation_as_reference>
+    </plugin>
+  </sensor>
+</gazebo>
 </robot>

Commit message: t

File: description/robot_core.xacro (robot description, xacro)
@@ -12,5 +12,5 @@
     <xacro:property name="wheel_offset_y" value="0.141"/>
     <xacro:property name="wheel_offset_z" value="0.01"/>
-    <xacro:property name="caster_wheel_radius" value="0.015"/>
+    <xacro:property name="caster_wheel_radius" value="0.016"/>
     <xacro:property name="caster_wheel_mass" value="0.01"/>
     <xacro:property name="caster_wheel_offset_x" value="0.215"/>

File: description/ros2_control.xacro (robot description, xacro)
@@ -8,8 +8,8 @@
                 <param name="right_wheel_name">right_wheel_joint</param>
                 <param name="loop_rate">30</param>
-                <param name="device">/dev/ttyUSB0</param>
+                <param name="device">/dev/ttyACM0</param>
                 <param name="baud_rate">115200</param>
                 <param name="timeout_ms">1000</param>
-                <param name="enc_counts_per_rev">989</param>
+                <param name="enc_counts_per_rev">1977</param>
             </hardware>
             <joint name="left_wheel_joint">
